Commit message: latest update, change gripper orientation, yaml files

File: src/bimanual_ur10e/config/gripper1_standalone.urdf.xacro (robot description, xacro)
@@ -10,4 +10,5 @@
     parent="world"
     child="gripper1_tool0_adapter"/>
+  <!-- right gripper -->
   <xacro:robotiq_gripper
     name="gripper1"

File: src/bimanual_ur10e/config/gripper2_standalone.urdf.xacro (robot description, xacro)
@@ -10,4 +10,5 @@
     parent="world"
     child="gripper2_tool0_adapter"/>
+  <!-- left gripper -->
   <xacro:robotiq_gripper
     name="gripper2"

File: src/bimanual_ur10e/urdf/bimanual_ur10e.urdf.xacro (robot description, xacro)
@@ -22,5 +22,5 @@
   <!-- Shared world link -->
   <link name="world"/>
-  <!-- ===== Robot 1 - left arm ===== -->
+  <!-- ===== Robot 1 - right arm ===== -->
   <xacro:ur_robot
     name="robot1"
@@ -38,5 +38,5 @@
     <origin xyz="0.7 0.0 0.0" rpy="0 0 ${-pi/3}"/>
   </xacro:ur_robot>
-  <!-- ===== Robot 2 - RIGHT arm ===== -->
+  <!-- ===== Robot 2 - left arm ===== -->
   <xacro:ur_robot
     name="robot2"
@@ -76,5 +76,5 @@
     use_fake_hardware="false"
     com_port="/dev/ttyUSB1">
-    <origin xyz="0 0 0" rpy="0 0 0"/>
+    <origin xyz="0 0 0" rpy="0 0 ${pi/2}"/>
   </xacro:robotiq_gripper>
 </robot>
